Commit message: 优化多摄像头融合节点，添加参数文件支持，改进TF等待机制，增强错误处理和调试信息，更新URDF描述以支持固定基座和双摄像头结构

File: src/rm_robot_description/urdf/rm_gimbal.urdf.xacro (robot description, xacro)
@@ -5,4 +5,10 @@
   <xacro:arg name="rpy" default="0 0 0" />
   <link name="odom" />
+  <!-- Base link fixed to odom: provide the expected 'base_link' frame for other nodes -->
+  <link name="base_link" />
+  <joint name="odom_to_base_link" type="fixed">
+    <parent link="odom" />
+    <child link="base_link" />
+  </joint>
   <link name="gimbal_link" />
   <joint name="gimbal_joint" type="floating">
@@ -11,7 +17,9 @@
   </joint>
   <link name="camera_link" />
+  <!-- Attach the camera to base_link for the fixed test cameras. If you want the camera to be
+       mounted on the gimbal, change parent back to 'gimbal_link'. -->
   <joint name="camera_joint" type="fixed">
     <origin xyz="$(arg xyz)" rpy="$(arg rpy)" />
-    <parent link="gimbal_link" />
+    <parent link="base_link" />
     <child link="camera_link" />
     <axis xyz="0 0 0" />

File: src/rm_robot_description/urdf/test_dual_camera.urdf.xacro (robot description, xacro)
@@ -1,10 +1,33 @@
 <?xml version="1.0"?>
 <!--
-Simple dual-camera test URDF xacro.
-Provides two camera links and frames for use in testing fusion/detector nodes.
+Dual-camera test URDF xacro.
+Structure:
+  odom (root)
+    ├── base_link (fixed joint: odom_to_base_link)
+    │   ├── camera_left_link (fixed)
+    │   │   └── camera_left_optical_frame
+    │   │       └── camera_left_visual
+    │   └── camera_right_link (fixed)
+    │       └── camera_right_optical_frame
+    │           └── camera_right_visual
+    └── gimbal_link (floating joint: odom_to_gimbal)
+        [预留用于未来的自瞄相机]
 -->
 <robot xmlns:xacro="http://www.ros.org/wiki/xacro" name="test_dual_camera">
-  <!-- Base link (could be base_link) -->
+  <!-- Root link (world/odom frame) -->
+  <link name="odom" />
+  <!-- Base link: main platform, fixed to odom -->
   <link name="base_link" />
+  <joint name="odom_to_base_link" type="fixed">
+    <parent link="odom" />
+    <child link="base_link" />
+    <origin xyz="0.0 0.0 0.0" rpy="0 0 0" />
+  </joint>
+  <!-- Gimbal link: movable platform for future auto-aim camera -->
+  <link name="gimbal_link" />
+  <joint name="gimbal_joint" type="floating">
+    <parent link="odom" />
+    <child link="gimbal_link" />
+  </joint>
   <!-- Left camera mount -->
   <link name="camera_left_link" />

Commit message: 修复 getCurrentPridection 方法中的状态预测计算，更新视频播放器参数配置，调整 gimbal 关节的父链接，启用视频播放功能，添加视频播放器节点配置

File: src/rm_robot_description/urdf/rm_gimbal.urdf.xacro (robot description, xacro)
@@ -21,5 +21,5 @@
   <joint name="camera_joint" type="fixed">
     <origin xyz="$(arg xyz)" rpy="$(arg rpy)" />
-    <parent link="base_link" />
+    <parent link="gimbal_link" />
     <child link="camera_link" />
     <axis xyz="0 0 0" />
