Commit message: feat: 第二个补盲相机

File: src/rm_robot_description/urdf/rm_gimbal_with_blind_camera.urdf.xacro (robot description, xacro)
@@ -9,7 +9,9 @@
   <xacro:arg name="main_camera_xyz" default="0.174275 0.000 0.086463" />
   <xacro:arg name="main_camera_rpy" default="0.0 0.1396 -0.00" />
-  <!-- Blind camera pose (symmetric with main camera, from usb_camera_driver config) -->
+  <!-- Blind camera pose (from usb_camera_driver config) -->
   <xacro:arg name="blind_camera_1_xyz" default="-0.175 0.0 0.086" />
   <xacro:arg name="blind_camera_1_rpy" default="0.0 0.14 ${pi}" />
+  <xacro:arg name="blind_camera_2_xyz" default="-0.1 -0.1 0.05" />
+  <xacro:arg name="blind_camera_2_rpy" default="0.0 0.14 ${pi/2}" />
   <link name="odom" />
   <!-- Base link fixed to odom -->
@@ -51,3 +53,16 @@
     <child link="blind_camera_1_optical_frame" />
   </joint>
+  <!-- Blind camera 2 -->
+  <link name="blind_camera_2_link" />
+  <joint name="blind_camera_2_joint" type="fixed">
+    <origin xyz="$(arg blind_camera_2_xyz)" rpy="$(arg blind_camera_2_rpy)" />
+    <parent link="gimbal_link" />
+    <child link="blind_camera_2_link" />
+  </joint>
+  <link name="blind_camera_2_optical_frame" />
+  <joint name="blind_camera_2_optical_joint" type="fixed">
+    <origin xyz="0 0 0" rpy="${-pi/2} 0 ${-pi/2}" />
+    <parent link="blind_camera_2_link" />
+    <child link="blind_camera_2_optical_frame" />
+  </joint>
 </robot>

Commit message: feat: 双补盲可行

File: src/rm_robot_description/urdf/rm_gimbal_with_blind_camera.urdf.xacro (robot description, xacro)
@@ -12,4 +12,6 @@
   <xacro:arg name="blind_camera_1_xyz" default="-0.175 0.0 0.086" />
   <xacro:arg name="blind_camera_1_rpy" default="0.0 0.14 ${pi}" />
+  <xacro:arg name="blind_camera_2_xyz" default="-0.175 0.05 0.086" />
+  <xacro:arg name="blind_camera_2_rpy" default="0.0 0.14 ${pi/2}" />
   <link name="odom" />
   <!-- Base link fixed to odom -->
@@ -51,3 +53,16 @@
     <child link="blind_camera_1_optical_frame" />
   </joint>
+  <!-- Blind camera 2 -->
+  <link name="blind_camera_2_link" />
+  <joint name="blind_camera_2_joint" type="fixed">
+    <origin xyz="$(arg blind_camera_2_xyz)" rpy="$(arg blind_camera_2_rpy)" />
+    <parent link="gimbal_link" />
+    <child link="blind_camera_2_link" />
+  </joint>
+  <link name="blind_camera_2_optical_frame" />
+  <joint name="blind_camera_2_optical_joint" type="fixed">
+    <origin xyz="0 0 0" rpy="${-pi/2} 0 ${-pi/2}" />
+    <parent link="blind_camera_2_link" />
+    <child link="blind_camera_2_optical_frame" />
+  </joint>
 </robot>

Commit message: feat: 三补盲

File: src/rm_robot_description/urdf/rm_gimbal_with_blind_camera.urdf.xacro (robot description, xacro)
@@ -14,4 +14,6 @@
   <xacro:arg name="blind_camera_2_xyz" default="-0.175 0.05 0.086" />
   <xacro:arg name="blind_camera_2_rpy" default="0.0 0.14 ${pi/2}" />
+  <xacro:arg name="blind_camera_3_xyz" default="-0.175 -0.05 0.086" />
+  <xacro:arg name="blind_camera_3_rpy" default="0.0 0.14 ${-pi/2}" />
   <link name="odom" />
   <!-- Base link fixed to odom -->
@@ -66,3 +68,16 @@
     <child link="blind_camera_2_optical_frame" />
   </joint>
+  <!-- Blind camera 3 -->
+  <link name="blind_camera_3_link" />
+  <joint name="blind_camera_3_joint" type="fixed">
+    <origin xyz="$(arg blind_camera_3_xyz)" rpy="$(arg blind_camera_3_rpy)" />
+    <parent link="gimbal_link" />
+    <child link="blind_camera_3_link" />
+  </joint>
+  <link name="blind_camera_3_optical_frame" />
+  <joint name="blind_camera_3_optical_joint" type="fixed">
+    <origin xyz="0 0 0" rpy="${-pi/2} 0 ${-pi/2}" />
+    <parent link="blind_camera_3_link" />
+    <child link="blind_camera_3_optical_frame" />
+  </joint>
 </robot>
